File: MicroUSB5vAndUSBUART.kicad_sch (KiCad schematic)
At the start: 18 parts, among them Q1 Q_NPN_BCE, Q2 Q_NPN_BCE, U2 USB_CON8, U3 CP2102N

Commit message: Vertical Horizontal Traces
Parts:
- added D13: D_Zener_Small_ALT, Diode_SMD:D_0603_1608Metric, symbol Device:D_Zener_Small_ALT
- Q1, Q2: footprint SparkfunSilicon-Standard:SOT23-5 -> Package_TO_SOT_SMD:SOT-23
- R2, R3, R4, R5, R6, R7, R8, R9: footprint Resistor_SMD:R_0603_1608Metric -> Resistor_SMD:R_0603_1608Metric_Pad0.98x0.95mm_HandSolder
Connections:
- net +5V: now also D13.1 (K)
- net VBUS: no longer D3.2 (A2), D6.2 (A), U2.1 (VBUS)
- new net: D3.2 (A2), D6.2 (A), U2.1 (+5V)
- new net Barrel Jack Input: D13.2 (A)
Changed lines of the file:
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@@
   (junction (at 22.86 40.64) (diameter 1.016) (color 0 0 0 0))
   (junction (at 22.86 114.3) (diameter 1.016) (color 0 0 0 0))
-  (junction (at 25.4 137.16) (diameter 1.016) (color 0 0 0 0))
+  (junction (at 25.4 137.16) (diameter 0) (color 0 0 0 0))
   (junction (at 33.02 58.42) (diameter 1.016) (color 0 0 0 0))
   (junction (at 35.56 114.3) (diameter 1.016) (color 0 0 0 0))
@@
   (junction (at 48.26 114.3) (diameter 1.016) (color 0 0 0 0))
   (junction (at 50.8 25.4) (diameter 1.016) (color 0 0 0 0))
-  (junction (at 53.34 25.4) (diameter 1.016) (color 0 0 0 0))
   (junction (at 63.5 30.48) (diameter 1.016) (color 0 0 0 0))
+  (junction (at 73.66 25.4) (diameter 0) (color 0 0 0 0))
   (junction (at 76.2 35.56) (diameter 1.016) (color 0 0 0 0))
   (junction (at 154.94 88.9) (diameter 1.016) (color 0 0 0 0))
@@
   (no_connect (at 104.14 114.3))
   (no_connect (at 104.14 121.92))
+  (wire (pts (xy 15.24 137.16) (xy 25.4 137.16))
+    (stroke (width 0) (type default) (color 0 0 0 0))
+  )
   (wire (pts (xy 20.32 114.3) (xy 22.86 114.3))
     (stroke (width 0) (type solid) (color 0 0 0 0))
@@
     (stroke (width 0) (type solid) (color 0 0 0 0))
   )
-  (wire (pts (xy 25.4 137.16) (xy 25.4 132.08))
-    (stroke (width 0) (type solid) (color 0 0 0 0))
-  )
   (wire (pts (xy 25.4 137.16) (xy 25.4 139.7))
     (stroke (width 0) (type solid) (color 0 0 0 0))
@@
     (stroke (width 0) (type solid) (color 0 0 0 0))
   )
-  (wire (pts (xy 50.8 25.4) (xy 53.34 25.4))
+  (wire (pts (xy 50.8 25.4) (xy 63.5 25.4))
     (stroke (width 0) (type solid) (color 0 0 0 0))
   )
@@
     (stroke (width 0) (type solid) (color 0 0 0 0))
   )
-  (wire (pts (xy 53.34 25.4) (xy 63.5 25.4))
-    (stroke (width 0) (type solid) (color 0 0 0 0))
+  (wire (pts (xy 53.34 15.24) (xy 63.5 15.24))
+    (stroke (width 0) (type default) (color 0 0 0 0))
   )
   (wire (pts (xy 53.34 63.5) (xy 53.34 71.12))
@@
     (stroke (width 0) (type solid) (color 0 0 0 0))
   )
-  (wire (pts (xy 68.58 25.4) (xy 78.74 25.4))
+  (wire (pts (xy 68.58 15.24) (xy 73.66 15.24))
+    (stroke (width 0) (type default) (color 0 0 0 0))
+  )
+  (wire (pts (xy 68.58 25.4) (xy 73.66 25.4))
     (stroke (width 0) (type solid) (color 0 0 0 0))
   )
@@
     (stroke (width 0) (type solid) (color 0 0 0 0))
   )
+  (wire (pts (xy 73.66 15.24) (xy 73.66 25.4))
+    (stroke (width 0) (type default) (color 0 0 0 0))
+  )
+  (wire (pts (xy 73.66 25.4) (xy 78.74 25.4))
+    (stroke (width 0) (type solid) (color 0 0 0 0))
+  )
   (wire (pts (xy 76.2 35.56) (xy 76.2 38.1))
     (stroke (width 0) (type solid) (color 0 0 0 0))
@@
     (stroke (width 0) (type solid) (color 0 0 0 0))
   )
+  (global_label "VBUS" (shape input) (at 15.24 137.16 90) (fields_autoplaced)
+    (effects (font (size 1.27 1.27)) (justify left))
+    (property "Intersheet References" "${INTERSHEET_REFS}" (id 0) (at 15.1606 129.8483 90)
+      (effects (font (size 1.27 1.27)) (justify left) hide)
+    )
+  )
   (global_label "RI" (shape input) (at 38.1 83.82 180) (fields_autoplaced)
     (effects (font (size 1.27 1.27)) (justify right))
@@
     )
   )
-  (global_label "VBUS" (shape input) (at 48.26 25.4 90) (fields_autoplaced)
-    (effects (font (size 1.27 1.27)) (justify left))
-    (property "Intersheet References" "${INTERSHEET_REFS}" (id 0) (at 48.1806 18.1836 90)
-      (effects (font (size 1.27 1.27)) (justify left) hide)
+  (global_label "Barrel Jack Input" (shape input) (at 53.34 15.24 180) (fields_autoplaced)
+    (effects (font (size 1.27 1.27)) (justify right))
+    (property "Intersheet References" "${INTERSHEET_REFS}" (id 0) (at 34.2355 15.1606 0)
+      (effects (font (size 1.27 1.27)) (justify right) hide)
     )
   )
@@
     )
     (property "Datasheet" "" (id 3) (at 22.86 109.22 0)
-      (effects (font (size 1.27 1.27)) hide)
-    )
-    (pin "1")
-  )
-  (symbol (lib_id "power:VBUS") (at 25.4 132.08 0) (unit 1)
-    (in_bom yes) (on_board yes) (fields_autoplaced)
-    (property "Reference" "#PWR0110" (id 0) (at 25.4 135.89 0)
-      (effects (font (size 1.27 1.27)) hide)
-    )
-    (property "Value" "VBUS" (id 1) (at 25.4 128.4754 0))
-    (property "Footprint" "" (id 2) (at 25.4 132.08 0)
-      (effects (font (size 1.27 1.27)) hide)
-    )
-    (property "Datasheet" "" (id 3) (at 25.4 132.08 0)
-      (effects (font (size 1.27 1.27)) hide)
-    )
-    (pin "1")
-  )
-  (symbol (lib_id "power:VBUS") (at 53.34 25.4 0) (unit 1)
-    (in_bom yes) (on_board yes) (fields_autoplaced)
-    (property "Reference" "#PWR0111" (id 0) (at 53.34 29.21 0)
-      (effects (font (size 1.27 1.27)) hide)
-    )
-    (property "Value" "VBUS" (id 1) (at 53.34 21.7954 0))
-    (property "Footprint" "" (id 2) (at 53.34 25.4 0)
-      (effects (font (size 1.27 1.27)) hide)
-    )
-    (property "Datasheet" "" (id 3) (at 53.34 25.4 0)
       (effects (font (size 1.27 1.27)) hide)
     )
@@
     (pin "1")
   )
+  (symbol (lib_id "Device:D_Zener_Small_ALT") (at 66.04 15.24 180) (unit 1)
+    (in_bom yes) (on_board yes) (fields_autoplaced)
+    (property "Reference" "D13" (id 0) (at 66.04 10.3844 0))
+    (property "Value" "D_Zener_Small_ALT" (id 1) (at 66.04 13.1595 0)
+      (effects (font (size 1.27 1.27)) hide)
+    )
+    (property "Footprint" "Diode_SMD:D_0603_1608Metric" (id 2) (at 66.04 15.24 90)
+      (effects (font (size 1.27 1.27)) hide)
+    )
+    (property "Datasheet" "~" (id 3) (at 66.04 15.24 90)
+      (effects (font (size 1.27 1.27)) hide)
+    )
+    (pin "1")
+    (pin "2")
+  )
   (symbol (lib_id "Device:D_Zener_Small_ALT") (at 66.04 25.4 180) (unit 1)
     (in_bom yes) (on_board yes) (fields_autoplaced)
@@
       (effects (font (size 1.27 1.27)) (justify left))
     )
-    (property "Footprint" "Resistor_SMD:R_0603_1608Metric" (id 2) (at 31.75 138.938 90)
+    (property "Footprint" "Resistor_SMD:R_0603_1608Metric_Pad0.98x0.95mm_HandSolder" (id 2) (at 31.75 138.938 90)
       (effects (font (size 1.27 1.27)) hide)
     )
@@
     (property "Reference" "R3" (id 0) (at 40.132 143.51 90))
     (property "Value" "47.5k" (id 1) (at 38.1 143.51 90))
-    (property "Footprint" "Resistor_SMD:R_0603_1608Metric" (id 2) (at 36.322 143.51 90)
+    (property "Footprint" "Resistor_SMD:R_0603_1608Metric_Pad0.98x0.95mm_HandSolder" (id 2) (at 36.322 143.51 90)
       (effects (font (size 1.27 1.27)) hide)
     )
@@
     (property "Reference" "R4" (id 0) (at 58.928 140.97 90))
     (property "Value" "2k" (id 1) (at 60.96 140.97 90))
-    (property "Footprint" "Resistor_SMD:R_0603_1608Metric" (id 2) (at 62.738 140.97 90)
+    (property "Footprint" "Resistor_SMD:R_0603_1608Metric_Pad0.98x0.95mm_HandSolder" (id 2) (at 62.738 140.97 90)
       (effects (font (size 1.27 1.27)) hide)
     )
@@
     (property "Reference" "R5" (id 0) (at 78.232 140.97 90))
     (property "Value" "10k" (id 1) (at 76.2 140.97 90))
-    (property "Footprint" "Resistor_SMD:R_0603_1608Metric" (id 2) (at 74.422 140.97 90)
+    (property "Footprint" "Resistor_SMD:R_0603_1608Metric_Pad0.98x0.95mm_HandSolder" (id 2) (at 74.422 140.97 90)
       (effects (font (size 1.27 1.27)) hide)
     )
@@
     (property "Reference" "R8" (id 0) (at 148.59 28.0374 90))
     (property "Value" "0" (id 1) (at 148.59 30.8125 90))
-    (property "Footprint" "Resistor_SMD:R_0603_1608Metric" (id 2) (at 148.59 34.798 90)
+    (property "Footprint" "Resistor_SMD:R_0603_1608Metric_Pad0.98x0.95mm_HandSolder" (id 2) (at 148.59 34.798 90)
       (effects (font (size 1.27 1.27)) hide)
     )
@@
     (property "Reference" "R9" (id 0) (at 148.59 38.1974 90))
     (property "Value" "0" (id 1) (at 148.59 40.9725 90))
-    (property "Footprint" "Resistor_SMD:R_0603_1608Metric" (id 2) (at 148.59 44.958 90)
+    (property "Footprint" "Resistor_SMD:R_0603_1608Metric_Pad0.98x0.95mm_HandSolder" (id 2) (at 148.59 44.958 90)
       (effects (font (size 1.27 1.27)) hide)
     )
@@
     (property "Reference" "R7" (id 0) (at 163.83 83.9174 90))
     (property "Value" "10k" (id 1) (at 163.83 86.6925 90))
-    (property "Footprint" "Resistor_SMD:R_0603_1608Metric" (id 2) (at 163.83 90.678 90)
+    (property "Footprint" "Resistor_SMD:R_0603_1608Metric_Pad0.98x0.95mm_HandSolder" (id 2) (at 163.83 90.678 90)
       (effects (font (size 1.27 1.27)) hide)
     )
@@
     (property "Reference" "R6" (id 0) (at 163.83 104.2374 90))
     (property "Value" "10k" (id 1) (at 163.83 107.0125 90))
-    (property "Footprint" "Resistor_SMD:R_0603_1608Metric" (id 2) (at 163.83 110.998 90)
+    (property "Footprint" "Resistor_SMD:R_0603_1608Metric_Pad0.98x0.95mm_HandSolder" (id 2) (at 163.83 110.998 90)
       (effects (font (size 1.27 1.27)) hide)
     )
@@
       (effects (font (size 1.27 1.27)) (justify left))
     )
-    (property "Footprint" "SparkfunSilicon-Standard:SOT23-5" (id 2) (at 185.42 86.36 0)
+    (property "Footprint" "Package_TO_SOT_SMD:SOT-23" (id 2) (at 185.42 86.36 0)
       (effects (font (size 1.27 1.27)) hide)
     )
@@
       (effects (font (size 1.27 1.27)) (justify left))
     )
-    (property "Footprint" "SparkfunSilicon-Standard:SOT23-5" (id 2) (at 185.42 111.76 0)
-      (effects (font (size 1.27 1.27)) hide)
-    )
+    (property "Footprint" "Package_TO_SOT_SMD:SOT-23" (id 2) (at 185.42 111.76 0)
+      (effects (font (size 1.27 1.27)) hide)
+    )
