File: SensorModule.kicad_sch (KiCad schematic)
At the start: 9 parts, among them U6 ZMOD4410AI3V, U7 TSL2541

Commit message: Vertical Horizontal Traces
Parts:
- removed U7: TSL2541, symbol OpticalSensor:TSL2541
- added C13, C15, C16: 10u, Capacitor_SMD:C_0603_1608Metric, symbol Device:C
- added C14, C17: 0.1u, Capacitor_SMD:C_0603_1608Metric, symbol Device:C
- added C18: 1u, Capacitor_SMD:C_0603_1608Metric, symbol Device:C
- added D5, D7, D8, D9: LED, LED_SMD:LED_0603_1608Metric_Pad1.05x0.95mm_HandSolder, symbol Device:LED
- added JP1: Jumper, Jumper:SolderJumper-2_P1.3mm_Bridged_RoundedPad1.0x1.5mm, symbol Device:Jumper
- added R20, R21, R34, R35: 0, Resistor_SMD:R_0603_1608Metric_Pad0.98x0.95mm_HandSolder, symbol Device:R
- added R22, R23: 10k, Resistor_SMD:R_0603_1608Metric_Pad0.98x0.95mm_HandSolder, symbol Device:R
- added R24, R25, R27: 200, Resistor_SMD:R_0603_1608Metric_Pad0.98x0.95mm_HandSolder, symbol Device:R
- added U10: AT25SF041, Package_SO:SO-8_3.9x4.9mm_P1.27mm, symbol SparkFun-IC-Memory:AT25SF041
- added U7: AS72652, Package_LGA:AMS_LGA-20_4.7x4.5mm_P0.65mm, symbol Sensor_Optical:AS72651
- added U8: AS72651, Package_LGA:AMS_LGA-20_4.7x4.5mm_P0.65mm, symbol Sensor_Optical:AS72651
- added U9: AS72653, Package_LGA:AMS_LGA-20_4.7x4.5mm_P0.65mm, symbol Sensor_Optical:AS72651
- C12: value C -> 0.1u; footprint (none) -> Capacitor_SMD:C_0603_1608Metric
- R14, R15, R16: footprint (none) -> Resistor_SMD:R_0603_1608Metric_Pad0.98x0.95mm_HandSolder
- R17, R19: value R -> 2.2k; footprint (none) -> Resistor_SMD:R_0603_1608Metric_Pad0.98x0.95mm_HandSolder
- R18: value R -> 10k; footprint (none) -> Resistor_SMD:R_0603_1608Metric_Pad0.98x0.95mm_HandSolder
- U6: footprint (none) -> ZMOD4410-LGA-12_3x3:ZMOD4410-LGA-12_3x3
Connections:
- net +1V8 is gone; now on net +3V3: R19.2
- net SCA is gone; now on net +3V3: R18.1
- net +3V3: now also C12.2, R14.1, R15.1, R16.1, R17.1, C13.2, C14.2, C15.2, C16.2, C17.2, C18.2, D7.2 (A), R20.1, R21.1, R22.2, R23.2, U10.3 (~{WP(D2})), U10.7 (~{HOLD(D3})), U10.8 (VCC), U7.14 (VDD2), U7.17 (VDD1), U8.14 (VDD2), U8.17 (VDD1), U9.14 (VDD2), U9.17 (VDD1)
- net GND: now also C13.1, C14.1, C15.1, C16.1, C17.1, C18.1, JP1.1, U10.4 (GND), U7.16 (GND), U8.16 (GND), U9.16 (GND); no longer R14.1, R15.1
- net OpticalSensorInterrupt: now also U8.13 (INT); no longer R16.2
- net SCL: now also R21.2, U8.11 (RX/SCL_S); no longer R17.1
- net SDA: now also R20.2, U8.12 (TX/SDA_S)
- net AS72652AndAS72653_SDA: now reaches R19.1
- net AS72652AndAS72653_SDA: now also U7.10 (SDA_S), U8.10 (SDA_M), U9.10 (SDA_S); no longer C12.2
- removed net VBUS: R16.1, R17.2, R18.2
- new net: D5.1 (K), U7.15 (LED_DRV)
- new net: D5.2 (A), R24.1
- new net: R25.1, U8.15 (LED_DRV)
- new net: R35.1, U8.18 (LED_IND)
- new net: R16.2, R34.1, U8.8 (I2C_ENB)
- new net: D9.2 (A), R27.1
- new net: D8.1 (K), R25.2
- new net: D9.1 (K), U9.15 (LED_DRV)
- new net: JP1.2, R34.2
- new net: D7.1 (K), R35.2
- new net +5V: D8.2 (A), R24.2, R27.2
- new net AS72652AndAS72653_SCL: R17.2, U7.9 (SCL_S), U8.9 (SCL_M), U9.9 (SCL_S)
- new net OpticalSPICLK: U10.6 (SCK), U8.3 (SCK)
- new net OpticalSPIMISO: U10.2 (SO(D1)), U8.5 (MISO)
- new net OpticalSPIMOSI: U10.5 (SI(D0)), U8.4 (MOSI)
- new net OpticalSensorResetPin: R18.2, U8.2 (~{RES})
- new net SLV1Reset: U7.2 (~{RES})
- new net SLV1ResetPin: R22.1, U8.1 (~{SLV1_RES})
- new net SLV2Reset: U9.2 (~{RES})
- new net SLV2ResetPin: R23.1, U8.20 (~{SLV2_RES})
- new net ~{CS}: U10.1 (~{CS}), U8.6 (~{CS})
Other:
- note added: "Check into normally open/close symbol"
- moved on the sheet: C12, R16, R17, R18, R19
